Commit message: [add] 로봇 시각화 추가

File: assets/mobile_robot.urdf.xacro (robot description, xacro)
@@ -4,67 +4,72 @@
   <xacro:property name="wheel_radius" value="0.08"/>
   <xacro:property name="wheel_length" value="0.42"/> <!-- 바퀴 중심 간 거리 -->
-  <xacro:property name="base_size_x"  value="0.30"/> <!-- 박스 전체 폭(길이*2*size) -->
+  <xacro:property name="base_size_x"  value="0.30"/>
   <xacro:property name="base_size_y"  value="0.40"/>
   <xacro:property name="base_size_z"  value="0.10"/>
-  <link name="world"/>
-  <joint name="world_to_base" type="fixed">
-    <parent link="world"/>
-    <child link="base_link"/>
+  <!-- 관성 없는 루트(표준) -->
+  <link name="base_footprint"/>
+  <joint name="base_footprint_to_base_link" type="fixed">
+    <parent link="base_footprint"/>
+    <child  link="base_link"/>
+    <!-- 바닥 접점 기준으로 베이스가 바퀴 중심 높이에 오도록 -->
+    <origin xyz="0 0 ${wheel_radius}" rpy="0 0 0"/>
   </joint>
-  <!-- 링크: 베이스 -->
+  <!-- 베이스 -->
   <link name="base_link">
     <visual>
+      <origin xyz="0 0 0" rpy="0 0 0"/>
       <geometry><box size="${base_size_x} ${base_size_y} ${base_size_z}"/></geometry>
-      <material name="chassis_color">
-        <color rgba="0.2 0.2 0.25 1.0"/>
-      </material>
-      <origin xyz="0 0 ${wheel_radius - 0.03}" rpy="0 0 0"/>
+      <material name="chassis"><color rgba="0.2 0.2 0.25 1.0"/></material>
     </visual>
     <collision>
+      <origin xyz="0 0 0" rpy="0 0 0"/>
       <geometry><box size="${base_size_x} ${base_size_y} ${base_size_z}"/></geometry>
-      <origin xyz="0 0 ${wheel_radius - 0.03}" rpy="0 0 0"/>
     </collision>
     <inertial>
+      <origin xyz="0 0 0" rpy="0 0 0"/>
       <mass value="10.0"/>
       <inertia ixx="0.2" iyy="0.2" izz="0.2" ixy="0" ixz="0" iyz="0"/>
     </inertial>
   </link>
-  <!-- 왼쪽 바퀴 링크 -->
+  <!-- 왼쪽 바퀴 -->
   <link name="wheel_left_link">
     <visual>
+      <!-- 실린더 축(z)을 y축으로 회전 -->
+      <origin xyz="0 0 0" rpy="1.57079632679 0 0"/>
       <geometry><cylinder radius="${wheel_radius}" length="0.04"/></geometry>
-      <material name="wheel_color"><color rgba="0.1 0.1 0.1 1.0"/></material>
-      <origin xyz="0 ${wheel_length/2} ${wheel_radius}" rpy="0 0 0"/>
+      <material name="wheel"><color rgba="0.1 0.1 0.1 1.0"/></material>
     </visual>
     <collision>
+      <origin xyz="0 0 0" rpy="1.57079632679 0 0"/>
       <geometry><cylinder radius="${wheel_radius}" length="0.04"/></geometry>
-      <origin xyz="0 ${wheel_length/2} ${wheel_radius}" rpy="0 0 0"/>
     </collision>
     <inertial>
+      <origin xyz="0 0 0" rpy="0 0 0"/>
       <mass value="1.0"/>
       <inertia ixx="0.01" iyy="0.01" izz="0.01" ixy="0" ixz="0" iyz="0"/>
     </inertial>
   </link>
-  <!-- 오른쪽 바퀴 링크 -->
+  <!-- 오른쪽 바퀴 -->
   <link name="wheel_right_link">
     <visual>
+      <origin xyz="0 0 0" rpy="1.57079632679 0 0"/>
       <geometry><cylinder radius="${wheel_radius}" length="0.04"/></geometry>
-      <material name="wheel_color"/>
-      <origin xyz="0 ${-wheel_length/2} ${wheel_radius}" rpy="0 0 0"/>
+      <material name="wheel"/>
     </visual>
     <collision>
+      <origin xyz="0 0 0" rpy="1.57079632679 0 0"/>
       <geometry><cylinder radius="${wheel_radius}" length="0.04"/></geometry>
-      <origin xyz="0 ${-wheel_length/2} ${wheel_radius}" rpy="0 0 0"/>
     </collision>
     <inertial>
+      <origin xyz="0 0 0" rpy="0 0 0"/>
       <mass value="1.0"/>
       <inertia ixx="0.01" iyy="0.01" izz="0.01" ixy="0" ixz="0" iyz="0"/>
     </inertial>
   </link>
-  <!-- 힌지 회전축 = y축(로봇 오른쪽이 +y) -->
+  <!-- 힌지(y축 회전) : 바퀴 위치는 joint에서만 지정 -->
   <joint name="wheel_left_joint" type="continuous">
     <parent link="base_link"/>
     <child  link="wheel_left_link"/>
-    <origin xyz="0 ${wheel_length/2} ${wheel_radius}" rpy="0 0 0"/>
+    <origin xyz="0 ${wheel_length/2} 0" rpy="0 0 0"/>
     <axis xyz="0 1 0"/>
   </joint>
@@ -72,5 +77,5 @@
     <parent link="base_link"/>
     <child  link="wheel_right_link"/>
-    <origin xyz="0 ${-wheel_length/2} ${wheel_radius}" rpy="0 0 0"/>
+    <origin xyz="0 ${-wheel_length/2} 0" rpy="0 0 0"/>
     <axis xyz="0 1 0"/>
   </joint>

Commit message: [improve] 파라미터 변경

File: assets/mobile_robot.urdf.xacro (robot description, xacro)
@@ -2,6 +2,6 @@
 <robot name="mobile_robot" xmlns:xacro="http://www.ros.org/wiki/xacro">
   <!-- 파라미터 -->
-  <xacro:property name="wheel_radius" value="0.08"/>
-  <xacro:property name="wheel_length" value="0.42"/> <!-- 바퀴 중심 간 거리 -->
+  <xacro:property name="wheel_radius" value="0.065"/> <!-- Ø130mm/2 -->
+  <xacro:property name="wheel_length" value="0.4465"/> <!-- 바퀴 중심 간 거리 -->
   <xacro:property name="base_size_x"  value="0.30"/>
   <xacro:property name="base_size_y"  value="0.40"/>
